File: Front_End_Kicad/Front_End_Kicad.kicad_pcb (KiCad board)
At the start: 4 copper layers, 100 x 100 mm, 84 parts, among them J101 Barrel_Jack, J102 Conn_01x01_Male, J103 Conn_01x01_Male, J201 Conn_01x01_Male, J202 Barrel_Jack, J203 Conn_01x01_Male, SW101 SW_DIP_x02, SW102 SW_DIP_x02, SW103 SW_DIP_x05, SW104 SW_DIP_x05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

Commit message: PCB nearly complete.  Added schematics and layers
Parts:
- removed C103: 0.1uF, Capacitor_SMD:C_1206_3216Metric
- removed C202: 10uF, Capacitor_SMD:C_1206_3216Metric
- removed TP118: attn_5x_gnd, TestPoint:TestPoint_THTPad_1.5x1.5mm_Drill0.7mm
- removed TP120: attn_10x_gnd, TestPoint:TestPoint_THTPad_1.5x1.5mm_Drill0.7mm
- removed TP122: attn_20x_gnd, TestPoint:TestPoint_THTPad_1.5x1.5mm_Drill0.7mm
- moved TP103 175.0 mm to (230.0, 99.5), turned to 270 degrees
- moved TP102 169.5 mm to (230.0, 108.9), turned to 270 degrees
- moved C107 168.4 mm to (222.9, 98.2)
- moved R102 166.4 mm to (225.3, 98.2)
- moved U101 163.6 mm to (222.3, 104.3), turned to 270 degrees
- moved R101 161.1 mm to (225.2, 110.4), turned to 270 degrees
- moved R104 161.0 mm to (217.9, 101.9)
- moved TP105 160.6 mm to (212.5, 98.0), turned to 270 degrees
- moved R103 157.0 mm to (217.9, 106.7), turned to 0 degrees
- moved TP106 156.5 mm to (208.0, 96.5), turned to 270 degrees
- moved R106 155.7 mm to (213.1, 101.9), turned to 180 degrees
- moved TP108 151.8 mm to (204.0, 100.1), turned to 270 degrees
- moved R105 151.8 mm to (213.1, 106.7), turned to 0 degrees
- moved R107 149.6 mm to (209.2, 104.2), turned to 90 degrees
- moved TP104 147.1 mm to (212.5, 110.5), turned to 270 degrees
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Routing:
- net V_-5v: track 8.62 -> 126.0 mm, vias 0 -> 1
- net V_OFFSET: track 44.6 -> 88.6 mm, vias 0 -> 1
- net signal_attenuated: track 0.00 -> 41.8 mm
- net attenuation_1x_in: track 0.00 -> 36.9 mm
- net GND: track 43.8 -> 73.3 mm, vias 11 -> 19
- net attenuation_2x_out: track 2.00 -> 23.5 mm
- net attenuation_20x_out: track 2.20 -> 22.9 mm
- net attenuation_5x_in: track 2.22 -> 18.5 mm
- net signal_raw: track 2.54 -> 18.6 mm
- net attenuation_10x_in: track 2.20 -> 18.0 mm
- net V_SUPPLY_IN: track 12.5 -> 25.3 mm
- net signal_mode_selected: track 16.1 -> 27.4 mm
- net V_+5v: track 28.7 -> 39.7 mm, vias 0 -> 5
- net Net-(R102-Pad2): track 5.04 -> 15.1 mm
- net Net-(R101-Pad1): track 5.13 -> 15.1 mm
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Other:
- board size 100 x 100 mm -> 99.5 x 90.2 mm
- board text added: "+5V"
- board text added: "-5V"
- board text added: "-5V OFFSET +5V"
- board text added: "1"
- board text added: "10"
- board text added: "2"
- board text added: "20"
- board text added: "5"
- board text added: "AC"
- board text added: "DC"
- board text added: "GRAHAM MUELLER"
- board text added: "IN"
- board text added: "Mode Select"
- board text added: "OSU - SENIOR DESIGN 20201122 R1"
- board text added: "SCALE"

Commit message: Updated schematic
Changed lines of the file:
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@@
   (general
     (thickness 1.6)
-    (drawings 100)
+    (drawings 104)
     (tracks 327)
     (zones 0)
@@
   (layers
     (0 F.Cu signal)
-    (1 in1.Cu power hide)
-    (2 In2.Cu power hide)
-    (31 B.Cu signal hide)
-    (32 B.Adhes user)
-    (33 F.Adhes user)
-    (34 B.Paste user)
-    (35 F.Paste user)
-    (36 B.SilkS user)
-    (37 F.SilkS user)
-    (38 B.Mask user)
-    (39 F.Mask user)
-    (40 Dwgs.User user)
-    (41 Cmts.User user)
-    (42 Eco1.User user)
-    (43 Eco2.User user)
+    (1 in1.Cu power)
+    (2 In2.Cu power)
+    (31 B.Cu signal)
+    (32 B.Adhes user hide)
+    (33 F.Adhes user hide)
+    (34 B.Paste user hide)
+    (35 F.Paste user hide)
+    (36 B.SilkS user hide)
+    (37 F.SilkS user hide)
+    (38 B.Mask user hide)
+    (39 F.Mask user hide)
+    (40 Dwgs.User user hide)
+    (41 Cmts.User user hide)
+    (42 Eco1.User user hide)
+    (43 Eco2.User user hide)
     (44 Edge.Cuts user)
     (45 Margin user)
-    (46 B.CrtYd user)
-    (47 F.CrtYd user)
-    (48 B.Fab user)
+    (46 B.CrtYd user hide)
+    (47 F.CrtYd user hide)
+    (48 B.Fab user hide)
     (49 F.Fab user hide)
   )
   (setup
-    (last_trace_width 1)
+    (last_trace_width 0.25)
     (user_trace_width 0.25)
     (user_trace_width 0.5)
@@
     (aux_axis_origin 0 0)
     (grid_origin 198 147.5)
-    (visible_elements 7FFFFFFF)
+    (visible_elements 7FFDEF7F)
     (pcbplotparams
-      (layerselection 0x010f0_ffffffff)
+      (layerselection 0x030f0_ffffffff)
       (usegerberextensions false)
       (usegerberattributes false)
@@
       (psa4output false)
       (plotreference true)
-      (plotvalue true)
+      (plotvalue false)
       (plotinvisibletext false)
       (padsonsilk false)
@@
       (drillshape 0)
       (scaleselection 1)
-      (outputdirectory "Schematics/"))
+      (outputdirectory "Gerber/"))
   )
   (net 0 "")
@@
     (descr "10-lead though-hole mounted DIP package, row spacing 7.62 mm (300 mils)")
     (tags "THT DIP DIL PDIP 2.54mm 7.62mm 300mil")
-    (fp_text reference SW104 (at 3.81 -2.33 90) (layer F.SilkS)
+    (fp_text reference SW104 (at 3.81 -2.33 90) (layer F.SilkS) hide
       (effects (font (size 1 1) (thickness 0.15)))
     )
@@
     (tags capacitor)
     (attr smd)
-    (fp_text reference C106 (at 1.4 -3.4 90) (layer F.SilkS)
+    (fp_text reference C106 (at 4.2 -0.1 180) (layer F.SilkS)
       (effects (font (size 1 1) (thickness 0.15)))
     )
@@
     )
   )
+  (gr_line (start 165.5 27.5) (end 165.5 120) (layer Margin) (width 0.15))
+  (gr_line (start 270.5 27.5) (end 165.5 27.5) (layer Margin) (width 0.15))
+  (gr_line (start 270.5 120) (end 270.5 27.5) (layer Margin) (width 0.15))
+  (gr_line (start 165.5 120) (end 270.5 120) (layer Margin) (width 0.15))
   (gr_arc (start 223.3 61.4) (end 223.3 71.3) (angle -90) (layer F.SilkS) (width 0.3))
   (gr_line (start 178.7 71.3) (end 223.3 71.3) (layer F.SilkS) (width 0.3))
@@
     (min_thickness 0.254)
     (keepout (tracks allowed) (vias allowed) (copperpour not_allowed))
-    (fill (arc_segments 32) (thermal_gap 0.1) (thermal_bridge_width 0.508) (smoothing chamfer) (radius 1))
+    (fill (arc_segments 32) (thermal_gap 0.1) (thermal_bridge_width 0.508))
     (polygon
       (pts
@@
     (min_thickness 0.254)
     (keepout (tracks allowed) (vias allowed) (copperpour not_allowed))
-    (fill (arc_segments 32) (thermal_gap 0.1) (thermal_bridge_width 0.508) (smoothing chamfer) (radius 1))
+    (fill (arc_segments 32) (thermal_gap 0.1) (thermal_bridge_width 0.508))
     (polygon
       (pts
@@
     (min_thickness 0.254)
     (keepout (tracks allowed) (vias allowed) (copperpour not_allowed))
-    (fill (arc_segments 32) (thermal_gap 0.1) (thermal_bridge_width 0.508) (smoothing chamfer) (radius 1))
+    (fill (arc_segments 32) (thermal_gap 0.1) (thermal_bridge_width 0.508))
     (polygon
       (pts
