File: Front_End_Kicad/Front_End_Kicad.sch (KiCad schematic (older format))
At the start: 57 parts, among them J101 Barrel_Jack, J102 Conn_01x01_Male, J103 Conn_01x01_Male, SW101 SW_DIP_x02, SW102 SW_DIP_x02, SW103 SW_DIP_x05, SW104 SW_DIP_x05, U101 LMH6551MM

Commit message: PCB nearly complete.  Added schematics and layers
Parts:
- removed C103: 0.1uF, Capacitor_SMD:C_1206_3216Metric, symbol Device:C
- removed TP118: attn_5x_gnd, TestPoint:TestPoint_THTPad_1.5x1.5mm_Drill0.7mm, symbol Connector:TestPoint
- removed TP120: attn_10x_gnd, TestPoint:TestPoint_THTPad_1.5x1.5mm_Drill0.7mm, symbol Connector:TestPoint
- removed TP122: attn_20x_gnd, TestPoint:TestPoint_THTPad_1.5x1.5mm_Drill0.7mm, symbol Connector:TestPoint
- TP116: footprint TestPoint:TestPoint_2Pads_Pitch5.08mm_Drill1.3mm -> TestPoint:TestPoint_THTPad_1.5x1.5mm_Drill0.7mm
Other:
- moved on the sheet: C101, C102, C104, C105
Changed lines of the file:
@@
 L Device:C C104
 U 1 1 5FC5CA77
-P 2100 5700
-F 0 "C104" V 2352 5700 50  0000 C CNN
-F 1 "10uF" V 2261 5700 50  0000 C CNN
-F 2 "Capacitor_SMD:C_1206_3216Metric" H 2138 5550 50  0001 C CNN
-F 3 "~" H 2100 5700 50  0001 C CNN
-F 4 "https://www.digikey.com/en/products/detail/taiyo-yuden/EMK316BJ106KL-T/930691" H 2100 5700 50  0001 C CNN "part_url"
-	1    2100 5700
+P 1850 4150
+F 0 "C104" V 2102 4150 50  0000 C CNN
+F 1 "10uF" V 2011 4150 50  0000 C CNN
+F 2 "Capacitor_SMD:C_1206_3216Metric" H 1888 4000 50  0001 C CNN
+F 3 "~" H 1850 4150 50  0001 C CNN
+F 4 "https://www.digikey.com/en/products/detail/taiyo-yuden/EMK316BJ106KL-T/930691" H 1850 4150 50  0001 C CNN "part_url"
+	1    1850 4150
 	0    1    1    0
 $EndComp
@@
 L power:GND #PWR0102
 U 1 1 5FC8B79B
-P 1900 6200
-F 0 "#PWR0102" H 1900 5950 50  0001 C CNN
-F 1 "GND" H 1905 6027 50  0000 C CNN
-F 2 "" H 1900 6200 50  0001 C CNN
-F 3 "" H 1900 6200 50  0001 C CNN
-	1    1900 6200
+P 1650 4650
+F 0 "#PWR0102" H 1650 4400 50  0001 C CNN
+F 1 "GND" H 1655 4477 50  0000 C CNN
+F 2 "" H 1650 4650 50  0001 C CNN
+F 3 "" H 1650 4650 50  0001 C CNN
+	1    1650 4650
 	1    0    0    -1
 $EndComp
@@
 L Device:C C101
 U 1 1 5FC8B7A8
-P 1700 5700
-F 0 "C101" V 1952 5700 50  0000 C CNN
-F 1 "10uF" V 1861 5700 50  0000 C CNN
-F 2 "Capacitor_SMD:C_1206_3216Metric" H 1738 5550 50  0001 C CNN
-F 3 "~" H 1700 5700 50  0001 C CNN
-F 4 "https://www.digikey.com/en/products/detail/taiyo-yuden/EMK316BJ106KL-T/930691" H 1700 5700 50  0001 C CNN "part_url"
-	1    1700 5700
-	0    1    1    0
-$EndComp
-Wire Wire Line
-	1550 6100 1550 5700
-Text GLabel 1450 5700 0    50   Input ~ 0
+P 1450 4150
+F 0 "C101" V 1702 4150 50  0000 C CNN
+F 1 "10uF" V 1611 4150 50  0000 C CNN
+F 2 "Capacitor_SMD:C_1206_3216Metric" H 1488 4000 50  0001 C CNN
+F 3 "~" H 1450 4150 50  0001 C CNN
+F 4 "https://www.digikey.com/en/products/detail/taiyo-yuden/EMK316BJ106KL-T/930691" H 1450 4150 50  0001 C CNN "part_url"
+	1    1450 4150
+	0    1    1    0
+$EndComp
+Wire Wire Line
+	1300 4550 1300 4150
+Text GLabel 1200 4150 0    50   Input ~ 0
 V_+5v
-$Comp
-L Device:C C103
-U 1 1 5FCA3C5A
-P 1900 5350
-F 0 "C103" V 2152 5350 50  0000 C CNN
-F 1 "0.1uF" V 2061 5350 50  0000 C CNN
-F 2 "Capacitor_SMD:C_1206_3216Metric" H 1938 5200 50  0001 C CNN
-F 3 "~" H 1900 5350 50  0001 C CNN
-F 4 "https://www.digikey.com/en/products/detail/w%C3%BCrth-elektronik/885012208030/5453952" H 1900 5350 50  0001 C CNN "part_url"
-	1    1900 5350
-	0    1    1    0
-$EndComp
 Text GLabel 4350 1400 2    50   Input ~ 0
 attenuation_1x_in
@@
 Connection ~ 9450 1100
 $Comp
-L Connector:TestPoint TP116
-U 1 1 5FC58742
-P 9950 1850
-F 0 "TP116" H 9892 1876 50  0000 R CNN
-F 1 "attn_2x_gnd" H 9892 1967 50  0000 R CNN
-F 2 "TestPoint:TestPoint_2Pads_Pitch5.08mm_Drill1.3mm" H 10150 1850 50  0001 C CNN
-F 3 "~" H 10150 1850 50  0001 C CNN
-	1    9950 1850
-	-1   0    0    1
-$EndComp
-Connection ~ 9950 1850
-$Comp
 L Device:R R113
 U 1 1 5FC5AC6B
@@
 Connection ~ 9450 2550
 $Comp
-L Connector:TestPoint TP118
-U 1 1 5FC5AC97
-P 9950 3300
-F 0 "TP118" H 9892 3326 50  0000 R CNN
-F 1 "attn_5x_gnd" H 9892 3417 50  0000 R CNN
-F 2 "TestPoint:TestPoint_THTPad_1.5x1.5mm_Drill0.7mm" H 10150 3300 50  0001 C CNN
-F 3 "~" H 10150 3300 50  0001 C CNN
-	1    9950 3300
-	-1   0    0    1
-$EndComp
-Connection ~ 9950 3300
-$Comp
 L Device:R R114
 U 1 1 5FC781CE
@@
 	9450 3950 9300 3950
 $Comp
-L Connector:TestPoint TP120
-U 1 1 5FC781FA
-P 9950 4700
-F 0 "TP120" H 9892 4726 50  0000 R CNN
-F 1 "attn_10x_gnd" H 9892 4817 50  0000 R CNN
-F 2 "TestPoint:TestPoint_THTPad_1.5x1.5mm_Drill0.7mm" H 10150 4700 50  0001 C CNN
-F 3 "~" H 10150 4700 50  0001 C CNN
-	1    9950 4700
-	-1   0    0    1
-$EndComp
-Connection ~ 9950 4700
-$Comp
 L Device:R R115
 U 1 1 5FC8CA2A
@@
 Wire Wire Line
 	9450 5300 9300 5300
-$Comp
-L Connector:TestPoint TP122
-U 1 1 5FC8CA56
-P 9950 6050
-F 0 "TP122" H 9892 6076 50  0000 R CNN
-F 1 "attn_20x_gnd" H 9892 6167 50  0000 R CNN
-F 2 "TestPoint:TestPoint_THTPad_1.5x1.5mm_Drill0.7mm" H 10150 6050 50  0001 C CNN
-F 3 "~" H 10150 6050 50  0001 C CNN
-	1    9950 6050
-	-1   0    0    1
-$EndComp
-Connection ~ 9950 6050
 Wire Wire Line
 	2400 1600 2950 1600
@@
 	1100 1600 1300 1600
 Wire Wire Line
-	1900 5700 1900 6100
-Connection ~ 1550 5700
-Wire Wire Line
-	1450 5700 1550 5700
-Wire Wire Line
-	1850 6100 1900 6100
-Connection ~ 1900 6100
-Wire Wire Line
-	1900 6100 1900 6200
-Wire Wire Line
-	1950 6100 1900 6100
-Wire Wire Line
-	1950 5700 1900 5700
-Wire Wire Line
-	1850 5700 1900 5700
-Connection ~ 1900 5700
-Wire Wire Line
-	2250 5700 2350 5700
-Connection ~ 2250 5700
-Wire Wire Line
-	2250 5700 2250 6100
-Wire Wire Line
-	1750 5350 1550 5350
-Wire Wire Line
-	1550 5350 1550 5700
-Wire Wire Line
-	2050 5350 2250 5350
-Wire Wire Line
-	2250 5350 2250 5700
-Text Notes 1600 5200 0    50   ~ 0
-Buffer bypass
+	1650 4150 1650 4550
+Connection ~ 1300 4150
+Wire Wire Line
+	1200 4150 1300 4150
+Wire Wire Line
+	1600 4550 1650 4550
+Connection ~ 1650 4550
+Wire Wire Line
+	1650 4550 1650 4650
+Wire Wire Line
+	1700 4550 1650 4550
+Wire Wire Line
+	1700 4150 1650 4150
+Wire Wire Line
+	1600 4150 1650 4150
+Connection ~ 1650 4150
+Wire Wire Line
+	2000 4150 2100 4150
+Connection ~ 2000 4150
+Wire Wire Line
+	2000 4150 2000 4550
 Wire Wire Line
 	4550 3800 4550 4000
@@
 F1 "Front_End_Power.sch" 50
 $EndSheet
-Text GLabel 2350 5700 2    50   Input ~ 0
+Text GLabel 2100 4150 2    50   Input ~ 0
 V_-5v
 Wire Wire Line
@@
 L Device:C C102
 U 1 1 5FBB0AA3
-P 1700 6100
-F 0 "C102" V 1952 6100 50  0000 C CNN
-F 1 "0.1uF" V 1861 6100 50  0000 C CNN
-F 2 "Capacitor_SMD:C_1206_3216Metric" H 1738 5950 50  0001 C CNN
-F 3 "~" H 1700 6100 50  0001 C CNN
-F 4 "https://www.digikey.com/en/products/detail/w%C3%BCrth-elektronik/885012208030/5453952" H 1700 6100 50  0001 C CNN "part_url"
-	1    1700 6100
+P 1450 4550
+F 0 "C102" V 1702 4550 50  0000 C CNN
+F 1 "0.1uF" V 1611 4550 50  0000 C CNN
+F 2 "Capacitor_SMD:C_1206_3216Metric" H 1488 4400 50  0001 C CNN
+F 3 "~" H 1450 4550 50  0001 C CNN
+F 4 "https://www.digikey.com/en/products/detail/w%C3%BCrth-elektronik/885012208030/5453952" H 1450 4550 50  0001 C CNN "part_url"
+	1    1450 4550
 	0    1    1    0
 $EndComp
@@
 L Device:C C105
 U 1 1 5FBB44B5
-P 2100 6100
-F 0 "C105" V 2352 6100 50  0000 C CNN
-F 1 "0.1uF" V 2261 6100 50  0000 C CNN
-F 2 "Capacitor_SMD:C_1206_3216Metric" H 2138 5950 50  0001 C CNN
-F 3 "~" H 2100 6100 50  0001 C CNN
-F 4 "https://www.digikey.com/en/products/detail/w%C3%BCrth-elektronik/885012208030/5453952" H 2100 6100 50  0001 C CNN "part_url"
-	1    2100 6100
+P 1850 4550
+F 0 "C105" V 2102 4550 50  0000 C CNN
+F 1 "0.1uF" V 2011 4550 50  0000 C CNN
+F 2 "Capacitor_SMD:C_1206_3216Metric" H 1888 4400 50  0001 C CNN
+F 3 "~" H 1850 4550 50  0001 C CNN
+F 4 "https://www.digikey.com/en/products/detail/w%C3%BCrth-elektronik/885012208030/5453952" H 1850 4550 50  0001 C CNN "part_url"
+	1    1850 4550
 	0    1    1    0
 $EndComp
@@
 Wire Wire Line
 	7000 1600 7300 1600
+$Comp
+L Connector:TestPoint TP116
+U 1 1 5FF2EE3F
+P 9950 1850
+F 0 "TP116" H 9892 1876 50  0000 R CNN
+F 1 "attn_2x_gnd" H 9892 1967 50  0000 R CNN
+F 2 "TestPoint:TestPoint_THTPad_1.5x1.5mm_Drill0.7mm" H 10150 1850 50  0001 C CNN
+F 3 "~" H 10150 1850 50  0001 C CNN
+	1    9950 1850
+	-1   0    0    1
+$EndComp
+Text Notes 1350 3650 0    50   ~ 0
+Buffer bypass
 $EndSCHEMATC

Commit message: Added names to parts to show better
Parts:
- C101, C102, C104, C105, C106, C107, C108: part_name (none) -> Bypass Cap
- J102, J103: part_name (none) -> Male Header
- R101, R102, R103, R104, R105, R106, R107, R108, R109, R110, R111, R112, R113, R114, R115, R116, R117, R118, R119: part_name (none) -> Resistor
- U101: part_name (none) -> Fully Diff Op Amp
Changed lines of the file:
@@
 F 4 "Buffer" H 4650 4300 50  0001 C CNN "part_description"
 F 5 "https://www.digikey.com/en/products/detail/texas-instruments/LMH6551MM-NOPB/755058" H 4650 4300 50  0001 C CNN "part_url"
+F 6 "Fully Diff Op Amp" H 4650 4300 50  0001 C CNN "part_name"
 	1    4650 4300
 	1    0    0    -1
@@
 F 3 "~" H 4400 3500 50  0001 C CNN
 F 4 "https://www.digikey.com/en/products/detail/yageo/RC1206FR-07365RL/728844" V 4400 3500 50  0001 C CNN "part_url"
+F 5 "Resistor" H 4400 3500 50  0001 C CNN "part_name"
 	1    4400 3500
 	0    1    1    0
@@
 F 3 "~" H 1850 4150 50  0001 C CNN
 F 4 "https://www.digikey.com/en/products/detail/taiyo-yuden/EMK316BJ106KL-T/930691" H 1850 4150 50  0001 C CNN "part_url"
+F 5 "Bypass Cap" H 1850 4150 50  0001 C CNN "part_name"
 	1    1850 4150
 	0    1    1    0
@@
 F 3 "~" H 1450 4150 50  0001 C CNN
 F 4 "https://www.digikey.com/en/products/detail/taiyo-yuden/EMK316BJ106KL-T/930691" H 1450 4150 50  0001 C CNN "part_url"
+F 5 "Bypass Cap" H 1450 4150 50  0001 C CNN "part_name"
 	1    1450 4150
 	0    1    1    0
@@
 F 3 "~" H 9700 1400 50  0001 C CNN
 F 4 "https://www.digikey.com/en/products/detail/yageo/RC1206FR-0737R4L/728846" V 9700 1400 50  0001 C CNN "part_url"
+F 5 "Resistor" H 9700 1400 50  0001 C CNN "part_name"
 	1    9700 1400
 	0    1    1    0
@@
 F 3 "~" H 9450 1650 50  0001 C CNN
 F 4 "https://www.digikey.com/en/products/detail/stackpole-electronics-inc/RNCP1206FTD150R/2240318" V 9450 1650 50  0001 C CNN "part_url"
+F 5 "Resistor" H 9450 1650 50  0001 C CNN "part_name"
 	1    9450 1650
 	1    0    0    -1
@@
 F 3 "~" H 9700 2850 50  0001 C CNN
 F 4 "https://www.digikey.com/en/products/detail/stackpole-electronics-inc/RMCF1206JT120R/1757405" V 9700 2850 50  0001 C CNN "part_url"
+F 5 "Resistor" H 9700 2850 50  0001 C CNN "part_name"
 	1    9700 2850
 	0    1    1    0
@@
 F 3 "~" H 9450 3100 50  0001 C CNN
 F 4 "https://www.digikey.com/en/products/detail/stackpole-electronics-inc/RNCP1206FTD75R0/2240314" V 9450 3100 50  0001 C CNN "part_url"
+F 5 "Resistor" H 9450 3100 50  0001 C CNN "part_name"
 	1    9450 3100
 	1    0    0    -1
@@
 F 3 "~" H 9700 4250 50  0001 C CNN
 F 4 "https://www.digikey.com/en/products/detail/stackpole-electronics-inc/RNCP1206FTD249R/2240322" V 9700 4250 50  0001 C CNN "part_url"
+F 5 "Resistor" H 9700 4250 50  0001 C CNN "part_name"
 	1    9700 4250
 	0    1    1    0
@@
 F 3 "~" H 9450 4500 50  0001 C CNN
 F 4 "https://www.digikey.com/en/products/detail/stackpole-electronics-inc/RMCF1206FT60R4/1754118" V 9450 4500 50  0001 C CNN "part_url"
+F 5 "Resistor" H 9450 4500 50  0001 C CNN "part_name"
 	1    9450 4500
 	1    0    0    -1
@@
 F 3 "" H 9700 5600 50  0001 C CNN
 F 4 "https://www.digikey.com/en/products/detail/stackpole-electronics-inc/RNCP1206FTD499R/2240329" V 9700 5600 50  0001 C CNN "part_url"
+F 5 "Resistor" H 9700 5600 50  0001 C CNN "part_name"
 	1    9700 5600
 	0    1    1    0
@@
 F 3 "~" H 9450 5850 50  0001 C CNN
 F 4 "https://www.digikey.com/en/products/detail/panasonic-electronic-components/ERJ-8ENF54R9V/88616" V 9450 5850 50  0001 C CNN "part_url"
+F 5 "Resistor" H 9450 5850 50  0001 C CNN "part_name"
 	1    9450 5850
 	1    0    0    -1
@@
 F 3 "~" H 9950 1650 50  0001 C CNN
 F 4 "https://www.digikey.com/en/products/detail/stackpole-electronics-inc/RNCP1206FTD150R/2240318" V 9950 1650 50  0001 C CNN "part_url"
+F 5 "Resistor" H 9950 1650 50  0001 C CNN "part_name"
 	1    9950 1650
 	-1   0    0    1
@@
 F 3 "~" H 9950 3100 50  0001 C CNN
 F 4 "https://www.digikey.com/en/products/detail/stackpole-electronics-inc/RNCP1206FTD75R0/2240314" V 9950 3100 50  0001 C CNN "part_url"
+F 5 "Resistor" H 9950 3100 50  0001 C CNN "part_name"
 	1    9950 3100
 	-1   0    0    1
@@
 F 3 "~" H 9950 4500 50  0001 C CNN
 F 4 "https://www.digikey.com/en/products/detail/stackpole-electronics-inc/RMCF1206FT60R4/1754118" V 9950 4500 50  0001 C CNN "part_url"
+F 5 "Resistor" H 9950 4500 50  0001 C CNN "part_name"
 	1    9950 4500
 	-1   0    0    1
@@
 F 3 "~" H 9950 5850 50  0001 C CNN
 F 4 "https://www.digikey.com/en/products/detail/panasonic-electronic-components/ERJ-8ENF54R9V/88616" V 9950 5850 50  0001 C CNN "part_url"
+F 5 "Resistor" H 9950 5850 50  0001 C CNN "part_name"
 	1    9950 5850
 	-1   0    0    1
@@
 F 3 "~" H 2600 1700 50  0001 C CNN
 F 4 "https://www.digikey.com/en/products/detail/w%C3%BCrth-elektronik/885012208030/5453952" H 2600 1700 50  0001 C CNN "part_url"
+F 5 "Bypass Cap" H 2600 1700 50  0001 C CNN "part_name"
 	1    2600 1700
 	0    1    1    0
@@
 F 3 "~" H 3700 4450 50  0001 C CNN
 F 4 "https://www.digikey.com/en/products/detail/w%C3%BCrth-elektronik/885012208030/5453952" H 3700 4450 50  0001 C CNN "part_url"
+F 5 "Bypass Cap" H 3700 4450 50  0001 C CNN "part_name"
 	1    3700 4450
 	1    0    0    -1
@@
 F 3 "~" H 1450 4550 50  0001 C CNN
 F 4 "https://www.digikey.com/en/products/detail/w%C3%BCrth-elektronik/885012208030/5453952" H 1450 4550 50  0001 C CNN "part_url"
+F 5 "Bypass Cap" H 1450 4550 50  0001 C CNN "part_name"
 	1    1450 4550
 	0    1    1    0
@@
 F 3 "~" H 1850 4550 50  0001 C CNN
 F 4 "https://www.digikey.com/en/products/detail/w%C3%BCrth-elektronik/885012208030/5453952" H 1850 4550 50  0001 C CNN "part_url"
+F 5 "Bypass Cap" H 1850 4550 50  0001 C CNN "part_name"
 	1    1850 4550
 	0    1    1    0
@@
 F 3 "~" H 3900 4200 50  0001 C CNN
 F 4 "https://www.digikey.com/en/products/detail/yageo/RC1206FR-07365RL/728844" V 3900 4200 50  0001 C CNN "part_url"
+F 5 "Resistor" H 3900 4200 50  0001 C CNN "part_name"
 	1    3900 4200
 	0    1    1    0
@@
 F 3 "~" H 4400 4950 50  0001 C CNN
 F 4 "https://www.digikey.com/en/products/detail/yageo/RC1206FR-07365RL/728844" V 4400 4950 50  0001 C CNN "part_url"
+F 5 "Resistor" H 4400 4950 50  0001 C CNN "part_name"
 	1    4400 4950
 	0    -1   -1   0
@@
 F 3 "~" H 3900 4950 50  0001 C CNN
 F 4 "https://www.digikey.com/en/products/detail/yageo/RC1206FR-07365RL/728844" V 3900 4950 50  0001 C CNN "part_url"
+F 5 "Resistor" H 3900 4950 50  0001 C CNN "part_name"
 	1    3900 4950
 	0    -1   -1   0
@@
 F 3 "~" H 5850 4100 50  0001 C CNN
 F 4 "https://www.digikey.com/en/products/detail/stackpole-electronics-inc/RMCF1206FT60R4/1754118" V 5850 4100 50  0001 C CNN "part_url"
+F 5 "Resistor" H 5850 4100 50  0001 C CNN "part_name"
 	1    5850 4100
 	0    1    1    0
@@
 F 3 "~" H 5850 4500 50  0001 C CNN
 F 4 "https://www.digikey.com/en/products/detail/stackpole-electronics-inc/RMCF1206FT60R4/1754118" V 5850 4500 50  0001 C CNN "part_url"
+F 5 "Resistor" H 5850 4500 50  0001 C CNN "part_name"
 	1    5850 4500
 	0    -1   -1   0
@@
 F 3 "" H 6100 4300 50  0001 C CNN
 F 4 "https://www.digikey.com/en/products/detail/stackpole-electronics-inc/RNCP1206FTD499R/2240329" V 6100 4300 50  0001 C CNN "part_url"
+F 5 "Resistor" H 6100 4300 50  0001 C CNN "part_name"
 	1    6100 4300
 	1    0    0    -1
@@
 F 3 "~" H 6300 4300 50  0001 C CNN
 F 4 "https://www.digikey.com/en/products/detail/w%C3%BCrth-elektronik/885012008001/5453716" H 6300 4300 50  0001 C CNN "part_url"
+F 5 "Bypass Cap" H 6300 4300 50  0001 C CNN "part_name"
 	1    6300 4300
 	1    0    0    -1
@@
 F 2 "Connector_PinHeader_2.00mm:PinHeader_1x01_P2.00mm_Vertical" H 1300 800 50  0001 C CNN
 F 3 "~" H 1300 800 50  0001 C CNN
+F 4 "Male Header" H 1300 800 50  0001 C CNN "part_name"
 	1    1300 800
 	0    1    1    0
@@
 F 2 "Connector_PinHeader_2.00mm:PinHeader_1x01_P2.00mm_Vertical" H 1300 2100 50  0001 C CNN
 F 3 "~" H 1300 2100 50  0001 C CNN
+F 4 "Male Header" H 1300 2100 50  0001 C CNN "part_name"
 	1    1300 2100
 	0    -1   -1   0

Commit message: Updated schematic
Parts:
- J102: value Conn_01x01_Male -> Signal_raw_in
- J103: value Conn_01x01_Male -> Signal_gnd
Other:
- note added: "-5v to +5v power supply\n"
- note added: "Attenuation selection\n"
- note added: "DC or AC mode selection"
- note added: "Differential Opamp"
- note added: "Impedance selection"
- note added: "Load is 500ohms and a 10pF cap to partially simulate an ADC"
- note added: "Vcm is connected to the adjustable DC Offset"
- note added: "Z=50\nZin == Zout"
- note removed: "DC AC Selector\nSwitches clearly named"
- note removed: "R1 : L and R"
- note removed: "R1: -55.28 Ω\nR2: -497.6 Ω"
- note removed: "R1: -61.11 Ω\nR2: -247.5 Ω"
- note removed: "R1: -74.93 Ω\nR2: -120.3 Ω"
- note removed: "TEST PADS\nTEXT !!! especially for selectors\nand test points\n\nClear values used, text for what each area does.\n\nArt for impedance in VS impedance out?"
- note removed: "\nR1: -150.5 Ω\nR2: -37.35 Ω"
- moved on the sheet: C101, C102, C104, C105, C106, C107, C108, J101, J102, J103, R101, R102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
